File: ergogen/output/pcbs/right.kicad_pcb (KiCad board)
At the start: 2 copper layers, 140.9 x 102.2 mm, 49 parts

Commit message: Pre-Routing Commit
Parts:
- removed the ? at (86.8, 9.45)
- removed the ? at (28.0, -10.5)
- removed the ? at (10.0, -29.5)
- removed the ? at (66.0, -42.5)
- removed the ? at (48.0, -21.5)
- added ?: , HOLE_M2_TH, F.Cu at (181.2, 9.45)
- added ?: , HOLE_M2_TH, F.Cu at (240.0, -10.5)
- added ?: , HOLE_M2_TH, F.Cu at (258.0, -29.5)
- added ?: , HOLE_M2_TH, F.Cu at (202.0, -42.5)
- added ?: , HOLE_M2_TH, F.Cu at (220.0, -21.5)
- moved D1 268.0 mm to (259.8, -15.5), turned to -90 degrees
- moved S1 268.0 mm to (268.0, -19.0)
- moved S2 268.0 mm to (268.0, -38.0)
- moved D2 251.9 mm to (240.8, 3.50), turned to -90 degrees
- moved D3 233.1 mm to (240.8, -34.5), turned to -90 degrees
- moved S3 230.0 mm to (249.0, 0.00)
- moved S4 230.0 mm to (249.0, -19.0)
- moved S5 230.0 mm to (249.0, -38.0)
- moved D4 211.2 mm to (221.8, -5.50), turned to -90 degrees
- moved D5 192.9 mm to (221.8, -43.5), turned to -90 degrees
- moved S6 192.0 mm to (230.0, -9.00)
- moved S7 192.0 mm to (230.0, -28.0)
- moved S8 192.0 mm to (230.0, -47.0)
- moved D17 188.2 mm to (214.0, -42.5), turned to -180 degrees
- moved D16 187.9 mm to (198.8, -31.5), turned to -90 degrees
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Connections:
- net far_thumb renamed mirror_inner_home
- net home_thumb renamed mirror_inner_top
- net index_bottom renamed mirror_index_home
- net index_home renamed mirror_inner_bottom
- net index_top renamed mirror_pinky_home
- net inner_bottom renamed mirror_near_thumb
- net inner_home renamed mirror_home_thumb
- net inner_top renamed mirror_outer_top
- net middle_bottom renamed mirror_middle_home
- net middle_home renamed mirror_ring_home
- net middle_top renamed mirror_index_bottom
- net near_thumb renamed mirror_far_thumb
- net outer_home renamed mirror_outer_home
- net outer_top renamed mirror_pinky_bottom
- net pinky_bottom renamed mirror_pinky_top
- net pinky_home renamed mirror_ring_bottom
- net pinky_top renamed mirror_index_top
- net ring_bottom renamed mirror_middle_top
- net ring_home renamed mirror_ring_top
- net ring_top renamed mirror_middle_bottom
- D10 pad 1: P029 -> P002
- D11 pad 1: P002 -> P155
- D12 pad 1: P029 -> P155
- D14 pad 1: P155 -> P031
- D15 pad 1: P155 -> P029
- D17 pad 1: P002 -> P031
- D19 pad 1: P031 -> P029
- D2 pad 1: P031 -> P002
- D3 pad 1: P002 -> P031
- D4 pad 1: P029 -> P002
- D5 pad 1: P029 -> P031
- D6 pad 1: P031 -> P002
- D7 pad 1: P002 -> P029
- D8 pad 1: P031 -> P002
- D9 pad 1: P002 -> P029
Other:
- outline, holes or cut-outs redrawn
